Commit message: It kind of works and I'm too tired
I switched to a continuous control scheme using gaussian distribution as oposed to the discrete one. Also changed some things in the car urdf

File: isaac_training/rc_car.urdf (robot description, URDF)
Before this commit: robot rc_car, 5 links, 4 joints
Links:
- added link front_left_steer_link, mass 0.01
- added link front_right_steer_link, mass 0.01
Joints:
- added joint front_left_wheel_joint: type continuous, parent front_left_steer_link, child front_left_wheel, origin xyz=0 0 0 rpy=1.5708 0 0, axis 0 0 1
- added joint front_right_wheel_joint: type continuous, parent front_right_steer_link, child front_right_wheel, origin xyz=0 0 0 rpy=1.5708 0 0, axis 0 0 1
- joint front_left_steer_joint: child front_left_wheel -> front_left_steer_link; limit lower=-0.5 upper=0.5 effort=1.0 velocity=1.0 -> lower=-0.5 upper=0.5 effort=10.0 velocity=1.0; origin xyz=0.12 0.09 -0.03 rpy=1.5708 0 0 -> xyz=0.12 0.09 -0.03 rpy=0 0 0
- joint front_right_steer_joint: child front_right_wheel -> front_right_steer_link; limit lower=-0.5 upper=0.5 effort=1.0 velocity=1.0 -> lower=-0.5 upper=0.5 effort=10.0 velocity=1.0; origin xyz=0.12 -0.09 -0.03 rpy=1.5708 0 0 -> xyz=0.12 -0.09 -0.03 rpy=0 0 0
